File: THAT1512  INA128 input NEVIN v4.brd (EAGLE design)
At the start: 63.8 x 124.5 mm, 85 parts, among them U1 THAT1512SO8-U, U2 THAT1512SO8-U, U3 TL072D

Commit message: Fixed routing
Parts:
- moved R1 0.76 mm to (17.8, 71.0)
Routing:
- net +5V: track 298.7 -> 275.3 mm, vias 4 -> 3
- net VR1_S1: track 45.4 -> 49.2 mm
- net SENSE1: track 78.6 -> 78.1 mm, vias 3 -> 2
- net VR2_S2: track 57.2 -> 57.0 mm, vias 0 -> 1
Changed lines of the file:
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@@
 <attribute name="VALUE" x="-0.897" y="15.58" size="1.27" layer="27" rot="R180" align="center"/>
 </element>
-<element name="R1" library="rc-master-smd" package="R0805" value="470" x="17.78" y="70.231" smashed="yes" rot="R90">
-<attribute name="NAME" x="16.51" y="68.453" size="0.8128" layer="25" ratio="18" rot="R90"/>
-<attribute name="VALUE" x="19.558" y="68.453" size="0.6096" layer="27" ratio="10" rot="R90"/>
+<element name="R1" library="rc-master-smd" package="R0805" value="470" x="17.78" y="70.993" smashed="yes" rot="R90">
+<attribute name="NAME" x="16.51" y="69.215" size="0.8128" layer="25" ratio="18" rot="R90"/>
+<attribute name="VALUE" x="19.558" y="69.215" size="0.6096" layer="27" ratio="10" rot="R90"/>
 </element>
 <element name="R2" library="rc-master-smd" package="R0805" value="470" x="17.78" y="13.97" smashed="yes" rot="R90">
@@
 <via x="2.54" y="48.26" extent="1-16" drill="0.508"/>
 <via x="39.37" y="35.56" extent="1-16" drill="0.508"/>
-<via x="38.735" y="48.26" extent="1-16" drill="0.508"/>
+<via x="39.116" y="47.879" extent="1-16" drill="0.508"/>
 <via x="43.18" y="56.896" extent="1-16" drill="0.508"/>
 <via x="44.577" y="29.591" extent="1-16" drill="0.508"/>
@@
 <via x="33.02" y="105.918" extent="1-16" drill="0.508"/>
 <via x="52.705" y="63.119" extent="1-16" drill="0.508"/>
-<via x="47.244" y="48.26" extent="1-16" drill="0.508"/>
+<via x="47.244" y="48.006" extent="1-16" drill="0.508"/>
 <via x="51.689" y="52.07" extent="1-16" drill="0.508"/>
 <via x="50.546" y="80.772" extent="1-16" drill="0.508"/>
@@
 <via x="48.26" y="80.772" extent="1-16" drill="0.508"/>
 <via x="9.652" y="69.469" extent="1-16" drill="0.508"/>
-<via x="29.21" y="48.26" extent="1-16" drill="0.508"/>
-<via x="10.16" y="48.26" extent="1-16" drill="0.508"/>
+<via x="28.702" y="47.879" extent="1-16" drill="0.508"/>
+<via x="10.287" y="48.006" extent="1-16" drill="0.508"/>
 <via x="35.56" y="52.07" extent="1-16" drill="0.508"/>
 <via x="21.717" y="54.356" extent="1-16" drill="0.508"/>
@@
 <wire x1="15.367" y1="49.022" x2="62.103" y2="49.022" width="0.6096" layer="16"/>
 <wire x1="62.103" y1="50.292" x2="62.23" y2="50.292" width="0.6096" layer="16"/>
-<wire x1="13.848" y1="54.658" x2="14.229" y2="54.658" width="0.6096" layer="16"/>
-<wire x1="17.102" y1="57.531" x2="14.229" y2="54.658" width="0.6096" layer="16"/>
-<wire x1="17.102" y1="57.531" x2="19.558" y2="57.531" width="0.6096" layer="16"/>
-<wire x1="19.558" y1="57.531" x2="20.828" y2="58.801" width="0.6096" layer="16"/>
-<wire x1="21.844" y1="72.898" x2="20.828" y2="71.882" width="0.6096" layer="16"/>
-<wire x1="20.828" y1="71.882" x2="20.828" y2="58.801" width="0.6096" layer="16"/>
-<via x="21.844" y="72.898" extent="1-16" drill="0.508"/>
-<wire x1="21.844" y1="72.898" x2="21.844" y2="73.025" width="0.4064" layer="1"/>
 <wire x1="59.69" y1="67.31" x2="60.96" y2="67.31" width="1.016" layer="1"/>
 <wire x1="60.96" y1="67.31" x2="62.23" y2="66.04" width="1.016" layer="1"/>
@@
 <signal name="SENSE1">
 <contactref element="IN1" pad="SS"/>
-<via x="25.908" y="30.988" extent="1-16" drill="0.508"/>
-<wire x1="25.908" y1="30.988" x2="20.193" y2="30.988" width="0.4064" layer="16"/>
+<wire x1="27.178" y1="30.988" x2="20.193" y2="30.988" width="0.4064" layer="16"/>
 <wire x1="14.224" y1="36.957" x2="14.224" y2="38.9698" width="0.4064" layer="16"/>
 <wire x1="14.224" y1="38.9698" x2="14.2968" y2="39.0426" width="0.4064" layer="16"/>
 <wire x1="20.193" y1="30.988" x2="14.224" y2="36.957" width="0.4064" layer="16"/>
-<wire x1="26.289" y1="31.369" x2="25.908" y2="30.988" width="0.4064" layer="1"/>
-<wire x1="40.64" y1="45.72" x2="25.908" y2="30.988" width="0.4064" layer="16"/>
-<wire x1="40.64" y1="45.72" x2="53.34" y2="45.72" width="0.4064" layer="16"/>
+<wire x1="41.91" y1="45.72" x2="27.178" y2="30.988" width="0.4064" layer="16"/>
+<wire x1="41.91" y1="45.72" x2="53.34" y2="45.72" width="0.4064" layer="16"/>
 <contactref element="IO" pad="5"/>
 <wire x1="59.69" y1="69.85" x2="58.42" y2="69.85" width="0.4064" layer="16"/>
@@
 <wire x1="38.735" y1="69.215" x2="39.37" y2="69.85" width="0.4064" layer="1"/>
 <via x="39.37" y="69.85" extent="1-16" drill="0.508"/>
-<wire x1="39.37" y1="69.85" x2="29.845" y2="69.85" width="0.4064" layer="16"/>
-<wire x1="29.845" y1="69.85" x2="27.686" y2="72.009" width="0.4064" layer="16"/>
+<wire x1="39.37" y1="69.85" x2="39.243" y2="69.85" width="0.4064" layer="16"/>
+<wire x1="39.243" y1="69.85" x2="37.084" y2="72.009" width="0.4064" layer="16"/>
+<wire x1="37.084" y1="72.009" x2="27.686" y2="72.009" width="0.4064" layer="16"/>
 <via x="27.686" y="72.009" extent="1-16" drill="0.508"/>
 <wire x1="27.686" y1="72.009" x2="26.543" y2="73.152" width="0.4064" layer="1"/>
@@
 <contactref element="VR1" pad="4"/>
 <contactref element="R36" pad="1"/>
-<wire x1="11.47" y1="8.89" x2="22.86" y2="8.89" width="0.4064" layer="16"/>
+<wire x1="11.216" y1="12.767" x2="11.216" y2="9.612" width="0.4064" layer="16"/>
+<wire x1="11.216" y1="9.612" x2="11.938" y2="8.89" width="0.4064" layer="16"/>
+<wire x1="11.938" y1="8.89" x2="22.86" y2="8.89" width="0.4064" layer="16"/>
 <wire x1="22.86" y1="8.89" x2="31.75" y2="0" width="0.4064" layer="16"/>
 <wire x1="31.75" y1="0" x2="42.0601625" y2="0" width="0.4064" layer="16"/>
@@
 <wire x1="11.203" y1="12.78" x2="17.606" y2="12.78" width="0.4064" layer="1"/>
 <wire x1="17.606" y1="12.78" x2="17.78" y2="12.954" width="0.4064" layer="1"/>
-<wire x1="11.47" y1="8.89" x2="11.203" y2="12.78" width="0" layer="19" extent="16-16"/>
+<wire x1="11.203" y1="12.78" x2="11.216" y2="12.767" width="0.4064" layer="16"/>
 </signal>
 <signal name="VR1_S2">
@@
 <wire x1="36.195" y1="62.17" x2="36.195" y2="59.309" width="0.4064" layer="1"/>
 <via x="36.195" y="59.309" extent="1-16" drill="0.508"/>
-<wire x1="36.195" y1="59.309" x2="32.639" y2="59.309" width="0.4064" layer="16"/>
-<wire x1="32.639" y1="59.309" x2="23.495" y2="50.165" width="0.4064" layer="16"/>
-<wire x1="23.495" y1="50.165" x2="18.542" y2="50.165" width="0.4064" layer="16"/>
+<wire x1="36.195" y1="59.309" x2="33.02" y2="59.309" width="0.4064" layer="16"/>
+<wire x1="33.02" y1="59.309" x2="23.876" y2="50.165" width="0.4064" layer="16"/>
+<wire x1="23.876" y1="50.165" x2="18.542" y2="50.165" width="0.4064" layer="16"/>
 <via x="18.542" y="50.165" extent="1-16" drill="0.508"/>
 <wire x1="18.542" y1="50.165" x2="9.525" y2="50.165" width="0.4064" layer="1"/>
@@
 <contactref element="R5" pad="1"/>
 <contactref element="R1" pad="1"/>
-<wire x1="17.78" y1="69.215" x2="12.774" y2="69.215" width="0.4064" layer="1"/>
-<wire x1="12.774" y1="69.215" x2="11.203" y2="67.644" width="0.4064" layer="1"/>
+<wire x1="17.78" y1="69.977" x2="13.536" y2="69.977" width="0.4064" layer="1"/>
+<wire x1="13.536" y1="69.977" x2="11.203" y2="67.644" width="0.4064" layer="1"/>
 <wire x1="11.203" y1="67.644" x2="11.203" y2="66.882" width="0.4064" layer="1"/>
 <wire x1="11.203" y1="66.882" x2="11.203" y2="68.353" width="0.4064" layer="16"/>
@@
 <contactref element="C20" pad="+"/>
 <contactref element="R1" pad="2"/>
-<wire x1="11.203" y1="71.882" x2="13.335" y2="71.882" width="0.4064" layer="1"/>
-<wire x1="13.97" y1="71.247" x2="13.335" y2="71.882" width="0.4064" layer="1"/>
-<wire x1="13.97" y1="71.247" x2="17.78" y2="71.247" width="0.4064" layer="1"/>
+<wire x1="17.78" y1="72.009" x2="17.653" y2="71.882" width="0.4064" layer="1"/>
+<wire x1="17.653" y1="71.882" x2="11.203" y2="71.882" width="0.4064" layer="1"/>
 <wire x1="11.203" y1="71.882" x2="11.203" y2="85.117" width="0.4064" layer="16"/>
 <wire x1="11.203" y1="85.117" x2="13.716" y2="87.63" width="0.4064" layer="16"/>
 <wire x1="13.716" y1="87.63" x2="20.193" y2="87.63" width="0.4064" layer="16"/>
 <wire x1="20.193" y1="87.63" x2="22.733" y2="90.17" width="0.4064" layer="16"/>
-<wire x1="44.45" y1="90.17" x2="45.72" y2="91.44" width="0.4064" layer="16"/>
-<wire x1="22.733" y1="90.17" x2="44.45" y2="90.17" width="0.4064" layer="16"/>
-<wire x1="45.72" y1="91.44" x2="45.72" y2="91.44" width="0" layer="19" extent="1-16"/>
+<wire x1="22.733" y1="90.17" x2="42.291" y2="90.17" width="0.4064" layer="16"/>
+<via x="42.291" y="90.17" extent="1-16" drill="0.508"/>
+<wire x1="45.72" y1="91.44" x2="44.45" y2="90.17" width="0.4064" layer="1"/>
+<wire x1="44.45" y1="90.17" x2="42.291" y2="90.17" width="0.4064" layer="1"/>
 </signal>
 <signal name="VR2_3">

Commit message: improved component placement and labeling
Parts:
- moved C16 9.68 mm to (29.1, 59.6)
- moved C18 8.23 mm to (29.8, 80.1)
- moved R11 4.71 mm to (29.2, 73.2), turned to 180 degrees
- moved L2 3.44 mm to (23.9, 12.4)
- moved R1 2.80 mm to (20.6, 71.1), turned to 180 degrees
- moved R4 2.80 mm to (29.1, 55.0), turned to 180 degrees
- moved C15 2.54 mm to (28.7, 2.54)
- moved L3 2.47 mm to (20.4, 65.2), turned to 0 degrees
- moved R6 2.16 mm to (37.1, 55.0)
- moved C5 2.01 mm to (26.7, 65.9)
- moved C24 1.80 mm to (31.2, 65.4)
- moved R2 1.70 mm to (18.5, 12.4)
- moved C6 1.49 mm to (29.1, 11.7), turned to 90 degrees
- moved R19 1.27 mm to (45.6, 22.4)
- moved R22 1.27 mm to (49.9, 22.4)
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Routing:
- net TIP2: track 33.3 -> 23.5 mm
- net V48+: track 197.0 -> 204.4 mm
- net N$14: track 18.9 -> 13.3 mm
- net VR2_S1: track 56.0 -> 61.3 mm
- net VR1_3: track 70.5 -> 65.2 mm
- net N$6: track 9.01 -> 13.9 mm
- net N$10: track 26.3 -> 30.6 mm
- net PHANTOM1: track 14.5 -> 17.7 mm
- net N$9: track 20.2 -> 18.0 mm
- net VR1_S2: track 53.7 -> 55.8 mm
- net VR2_S2: track 57.0 -> 59.0 mm
- net PHANTOM2: track 61.3 -> 63.1 mm
- net N$29: track 46.8 -> 45.0 mm
- net -12V: track 238.8 -> 237.1 mm
- net VR2_1: track 63.8 -> 62.1 mm
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