File: THAT1512  INA128 input NEVIN v4.sch (EAGLE design)
At the start: 85 parts, among them U1 THAT1512SO8-U, U2 THAT1512SO8-U, U3 TL072D

Commit message: Improved notes
Other:
- note added: "Combo Input Board Phantom power THAT1512 (C) 2020 RWP"
- note added: "D1-4: BAV170VL very low reverse current twin diodes. may be substituted by similar components (Ir <= 100nA, Vr > 50V), or with BAT54S twin (half bridge) Schottky diodes (better protection, slightly higher noise)."
- note added: "SENSE 1 & 2 require inputs with pullup resistors. LEDs draw 5mA at 3.3V"
- note added: "TT Corp switch pots - SPST push on-off P901S series 5K"
- note removed: "Combo Input Board Phantom power THAT1512"
- note removed: "D1-4: BAV170VL very low reverse current diodes. may be substituted by similar components (Ir <= 100nA, Vr > 50V), or with BAT54S twin (half bridge) Schottky diodes (better protection, slightly higher noise)."
- moved on the sheet: C15, C19, C3, C5, R1, R12, R25, R26
